File: remote/remote.brd (EAGLE design)
At the start: 63 x 24 mm, 44 parts, among them IC1 ATMEGA168-MU, SW1 MF-SW-TACT-4.2MM, SW2 MF-SW-TACT-4.2MM, SW3 MF-SW-TACT-4.2MM, SW4 CT05-XXXX-J1, U2 NRF24L01SMD, Y1 16M, Y2 12MHz

Commit message: remote: drop unsused net
Connections:
- removed net XXX: IC1.25
Changed lines of the file:
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@@
 <wire x1="48.8" y1="12" x2="50.6" y2="12" width="0.2" layer="1"/>
-</signal>
-<signal name="XXX">
-<contactref element="IC1" pad="25"/>
 </signal>
 </signals>
